File: arduino-etc/pcb/BootLoader_ATmega32U4/bootloader1.brd (EAGLE design)
At the start: 100 x 80 mm, 8 parts, among them U1 ATTINY85-20P

Commit message: UPD: pcb
Parts:
- moved VCC1 34.5 mm to (85.1, 30.5)
- moved VCC 34.2 mm to (31.8, 33.0)
- moved D10 22.7 mm to (49.5, 33.0), turned to 180 degrees
- moved SV1 22.7 mm to (77.5, 17.8), flipped to the bottom
- moved SV2 22.7 mm to (77.5, 30.5), flipped to the bottom
- moved U1 22.7 mm to (77.5, 24.1), flipped to the bottom
- moved GND 20.9 mm to (31.8, 17.8)
- moved GND2 12.7 mm to (69.8, 17.8)
Connections:
- net N$10 renamed PB0
- net N$2 renamed PB2
- net N$3 renamed RESET
- net N$7 renamed PB1
- net N$8 renamed PB4
- net N$9 renamed PB3
Routing:
- net GND: track 71.1 -> 48.3 mm, vias 2 -> 1
- net PB2: track 27.9 -> 48.3 mm, vias 0 -> 1
- net PB0: track 45.7 -> 27.9 mm, vias 2 -> 1
- net +5V: track 58.4 -> 69.8 mm, vias 2 -> 1
- net RESET: track 43.2 -> 53.3 mm, vias 0 -> 1
- net PB1: vias 0 -> 1
