File: arduino-etc/ATTiny85/ATTiny85+CirleLEDs+CR2032/pcb4-SK6812/attiny85.sch (EAGLE design)
At the start: 13 parts, among them SW1 bat+, SW2 POWER

Commit message: FIX: pcb4-SK6812/
Parts:
- added C1, C2, C3, C4, C5: (no value), rcl:C-EUC2012
- added PAD33: PAD150X50, ytani1:PAD150X50
Connections:
- net BAT+: now also C1.1, C2.1, C3.1, C4.1, C5.1
- net GND: now also C1.2, C2.2, C3.2, C4.2, C5.2
Changed lines of the file:
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@@
 <part name="GND8" library="supply1" library_urn="urn:adsk.eagle:library:371" deviceset="GND" device=""/>
 <part name="GND4" library="supply1" library_urn="urn:adsk.eagle:library:371" deviceset="GND" device=""/>
+<part name="C1" library="rcl" library_urn="urn:adsk.eagle:library:334" deviceset="C-EU" device="C2012" package3d_urn="urn:adsk.eagle:package:23625/2"/>
+<part name="C2" library="rcl" library_urn="urn:adsk.eagle:library:334" deviceset="C-EU" device="C2012" package3d_urn="urn:adsk.eagle:package:23625/2"/>
+<part name="C3" library="rcl" library_urn="urn:adsk.eagle:library:334" deviceset="C-EU" device="C2012" package3d_urn="urn:adsk.eagle:package:23625/2"/>
+<part name="C4" library="rcl" library_urn="urn:adsk.eagle:library:334" deviceset="C-EU" device="C2012" package3d_urn="urn:adsk.eagle:package:23625/2"/>
+<part name="C5" library="rcl" library_urn="urn:adsk.eagle:library:334" deviceset="C-EU" device="C2012" package3d_urn="urn:adsk.eagle:package:23625/2"/>
+<part name="GND9" library="supply1" library_urn="urn:adsk.eagle:library:371" deviceset="GND" device=""/>
+<part name="GND10" library="supply1" library_urn="urn:adsk.eagle:library:371" deviceset="GND" device=""/>
+<part name="GND11" library="supply1" library_urn="urn:adsk.eagle:library:371" deviceset="GND" device=""/>
+<part name="GND12" library="supply1" library_urn="urn:adsk.eagle:library:371" deviceset="GND" device=""/>
+<part name="GND13" library="supply1" library_urn="urn:adsk.eagle:library:371" deviceset="GND" device=""/>
+<part name="PAD33" library="ytani1" deviceset="PAD" device="150X50"/>
 </parts>
 <sheets>
@@
 <attribute name="VALUE" x="96.52" y="7.62" size="1.778" layer="96"/>
 </instance>
-<instance part="GND4" gate="1" x="73.66" y="48.26" smashed="yes">
-<attribute name="VALUE" x="71.12" y="45.72" size="1.778" layer="96"/>
-</instance>
+<instance part="GND4" gate="1" x="73.66" y="50.8" smashed="yes">
+<attribute name="VALUE" x="71.12" y="48.26" size="1.778" layer="96"/>
+</instance>
+<instance part="C1" gate="G$1" x="30.48" y="43.18" smashed="yes">
+<attribute name="NAME" x="32.004" y="43.561" size="1.778" layer="95"/>
+<attribute name="VALUE" x="32.004" y="38.481" size="1.778" layer="96"/>
+</instance>
+<instance part="C2" gate="G$1" x="50.8" y="43.18" smashed="yes">
+<attribute name="NAME" x="52.324" y="43.561" size="1.778" layer="95"/>
+<attribute name="VALUE" x="52.324" y="38.481" size="1.778" layer="96"/>
+</instance>
+<instance part="C3" gate="G$1" x="71.12" y="43.18" smashed="yes">
+<attribute name="NAME" x="72.644" y="43.561" size="1.778" layer="95"/>
+<attribute name="VALUE" x="72.644" y="38.481" size="1.778" layer="96"/>
+</instance>
+<instance part="C4" gate="G$1" x="91.44" y="43.18" smashed="yes">
+<attribute name="NAME" x="92.964" y="43.561" size="1.778" layer="95"/>
+<attribute name="VALUE" x="92.964" y="38.481" size="1.778" layer="96"/>
+</instance>
+<instance part="C5" gate="G$1" x="111.76" y="43.18" smashed="yes">
+<attribute name="NAME" x="113.284" y="43.561" size="1.778" layer="95"/>
+<attribute name="VALUE" x="113.284" y="38.481" size="1.778" layer="96"/>
+</instance>
+<instance part="GND9" gate="1" x="30.48" y="35.56" smashed="yes">
+<attribute name="VALUE" x="27.94" y="33.02" size="1.778" layer="96"/>
+</instance>
+<instance part="GND10" gate="1" x="50.8" y="35.56" smashed="yes">
+<attribute name="VALUE" x="48.26" y="33.02" size="1.778" layer="96"/>
+</instance>
+<instance part="GND11" gate="1" x="71.12" y="35.56" smashed="yes">
+<attribute name="VALUE" x="68.58" y="33.02" size="1.778" layer="96"/>
+</instance>
+<instance part="GND12" gate="1" x="91.44" y="35.56" smashed="yes">
+<attribute name="VALUE" x="88.9" y="33.02" size="1.778" layer="96"/>
+</instance>
+<instance part="GND13" gate="1" x="111.76" y="35.56" smashed="yes">
+<attribute name="VALUE" x="109.22" y="33.02" size="1.778" layer="96"/>
+</instance>
+<instance part="PAD33" gate="G$1" x="19.05" y="114.3" smashed="yes"/>
 </instances>
 <busses>
@@
 <segment>
 <pinref part="SV2" gate="G$1" pin="3"/>
-<wire x1="76.2" y1="58.42" x2="73.66" y2="50.8" width="0.1524" layer="91"/>
+<wire x1="76.2" y1="58.42" x2="73.66" y2="53.34" width="0.1524" layer="91"/>
 <pinref part="GND4" gate="1" pin="GND"/>
+</segment>
+<segment>
+<pinref part="GND9" gate="1" pin="GND"/>
+<pinref part="C1" gate="G$1" pin="2"/>
+</segment>
+<segment>
+<pinref part="GND10" gate="1" pin="GND"/>
+<pinref part="C2" gate="G$1" pin="2"/>
+</segment>
+<segment>
+<pinref part="GND11" gate="1" pin="GND"/>
+<pinref part="C3" gate="G$1" pin="2"/>
+</segment>
+<segment>
+<pinref part="GND12" gate="1" pin="GND"/>
+<pinref part="C4" gate="G$1" pin="2"/>
+</segment>
+<segment>
+<pinref part="GND13" gate="1" pin="GND"/>
+<pinref part="C5" gate="G$1" pin="2"/>
 </segment>
 </net>
@@
 <wire x1="76.2" y1="60.96" x2="66.04" y2="60.96" width="0.1524" layer="91"/>
 <pinref part="SK1" gate="G$1" pin="VDD"/>
-<wire x1="27.94" y1="33.02" x2="27.94" y2="44.45" width="0.1524" layer="91"/>
+<wire x1="27.94" y1="33.02" x2="27.94" y2="45.72" width="0.1524" layer="91"/>
 <pinref part="SK5" gate="G$1" pin="VDD"/>
-<wire x1="27.94" y1="44.45" x2="48.26" y2="44.45" width="0.1524" layer="91"/>
-<wire x1="48.26" y1="44.45" x2="66.04" y2="44.45" width="0.1524" layer="91"/>
-<wire x1="66.04" y1="44.45" x2="68.58" y2="44.45" width="0.1524" layer="91"/>
-<wire x1="68.58" y1="44.45" x2="88.9" y2="44.45" width="0.1524" layer="91"/>
-<wire x1="88.9" y1="44.45" x2="109.22" y2="44.45" width="0.1524" layer="91"/>
-<wire x1="109.22" y1="44.45" x2="109.22" y2="33.02" width="0.1524" layer="91"/>
+<wire x1="27.94" y1="45.72" x2="30.48" y2="45.72" width="0.1524" layer="91"/>
+<wire x1="30.48" y1="45.72" x2="48.26" y2="45.72" width="0.1524" layer="91"/>
+<wire x1="48.26" y1="45.72" x2="50.8" y2="45.72" width="0.1524" layer="91"/>
+<wire x1="50.8" y1="45.72" x2="66.04" y2="45.72" width="0.1524" layer="91"/>
+<wire x1="66.04" y1="45.72" x2="68.58" y2="45.72" width="0.1524" layer="91"/>
+<wire x1="68.58" y1="45.72" x2="71.12" y2="45.72" width="0.1524" layer="91"/>
+<wire x1="71.12" y1="45.72" x2="88.9" y2="45.72" width="0.1524" layer="91"/>
+<wire x1="88.9" y1="45.72" x2="91.44" y2="45.72" width="0.1524" layer="91"/>
+<wire x1="91.44" y1="45.72" x2="109.22" y2="45.72" width="0.1524" layer="91"/>
+<wire x1="109.22" y1="45.72" x2="109.22" y2="33.02" width="0.1524" layer="91"/>
 <pinref part="SK4" gate="G$1" pin="VDD"/>
-<wire x1="88.9" y1="33.02" x2="88.9" y2="44.45" width="0.1524" layer="91"/>
-<junction x="88.9" y="44.45"/>
+<wire x1="88.9" y1="33.02" x2="88.9" y2="45.72" width="0.1524" layer="91"/>
+<junction x="88.9" y="45.72"/>
 <pinref part="SK3" gate="G$1" pin="VDD"/>
-<wire x1="68.58" y1="33.02" x2="68.58" y2="44.45" width="0.1524" layer="91"/>
-<junction x="68.58" y="44.45"/>
+<wire x1="68.58" y1="33.02" x2="68.58" y2="45.72" width="0.1524" layer="91"/>
+<junction x="68.58" y="45.72"/>
 <pinref part="SK2" gate="G$1" pin="VDD"/>
-<wire x1="48.26" y1="33.02" x2="48.26" y2="44.45" width="0.1524" layer="91"/>
-<junction x="48.26" y="44.45"/>
-<wire x1="66.04" y1="60.96" x2="66.04" y2="44.45" width="0.1524" layer="91"/>
+<wire x1="48.26" y1="33.02" x2="48.26" y2="45.72" width="0.1524" layer="91"/>
+<junction x="48.26" y="45.72"/>
+<wire x1="66.04" y1="60.96" x2="66.04" y2="45.72" width="0.1524" layer="91"/>
 <junction x="66.04" y="60.96"/>
-<junction x="66.04" y="44.45"/>
-</segment>
-</net>
+<junction x="66.04" y="45.72"/>
+<pinref part="C1" gate="G$1" pin="1"/>
+<junction x="30.48" y="45.72"/>
+<pinref part="C2" gate="G$1" pin="1"/>
+<junction x="50.8" y="45.72"/>
+<pinref part="C3" gate="G$1" pin="1"/>
+<junction x="71.12" y="45.72"/>
+<pinref part="C4" gate="G$1" pin="1"/>
+<junction x="91.44" y="45.72"/>
+<pinref part="C5" gate="G$1" pin="1"/>
+<wire x1="111.76" y1="45.72" x2="109.22" y2="45.72" width="0.1524" layer="91"/>
+<junction x="109.22" y="45.72"/>
+</segment>
+</net>
