File: arduino-etc/ATTiny85/LedBadge/pcb/pcb2-SK6812/attiny85.sch (EAGLE design)
At the start: 19 parts, among them SW1 bat+, SW2 POWER

Commit message: UPD: pcb2-SK6812/
Parts:
- removed BAT+: bat+, ytani1:PINHEAD-MA01-1
- removed BAT-: bat-, ytani1:PINHEAD-MA01-1
- removed SV1: PIN-A, ytani1:PINHEAD-MA03-1
- removed SV2: PIN-B, ytani1:PINHEAD-MA03-1
- removed SW1: bat+, ytani1:PINHEAD-MA03-1
- added BAT1: (no value), ytani1:BAT-CR2032
- added H1, H2: (no value), ytani1:PINHEAD-MA03-1SMD
- added H3: (no value), ytani1:PINHEAD-MA03-1
- PAD33: value PAD150X50 -> PAD12X4; device ytani1:PAD150X50 -> ytani1:PAD12X4
Connections:
- net +3V3: now also BAT1.BAT+; no longer BAT+.1
- net BAT+: now also H2.2; no longer SV2.2
- net GND: now also BAT1.P$1, H2.3, H3.1; no longer BAT-.1, SV2.3, SW1.1, SW1.2
- net N$2: now also H2.1; no longer SV2.1
- net N$3: now also H1.3; no longer SV1.3
- net N$4: now also H1.1; no longer SV1.1
- net N$5: now also H1.2; no longer SV1.2
- net PB3: now also H3.3; no longer SW1.3
