File: arduino-etc/ATTiny85/LedBadge/pcb/pcb4-SK6812/attiny85.brd (EAGLE design)
At the start: 32 x 32 mm, 17 parts, among them SW2 POWER

Commit message: ADD: pcb4-SK6812/
Parts:
- removed SW2: POWER, ytani1:SW3-1
- added ON/OFF: POWER, ytani1:SW3-1
- BAT1: device ytani1:BAT-CR2032-2 -> ytani1:BAT-CR2032-3
- moved NP5 47.1 mm to (11.4, 25.4), turned to 270 degrees
- moved NP4 30.1 mm to (25.4, 11.4), turned to 0 degrees
- moved H3 25.4 mm to (12.7, 35.6), turned to 235 degrees
- moved C4 14.8 mm to (25.4, 15.2), turned to 0 degrees
- moved H2 11.4 mm to (22.9, 35.6)
- moved H1 11.4 mm to (30.5, 35.6)
- moved C3 11.1 mm to (35.6, 25.4)
- moved NP2 10.9 mm to (25.4, 39.4), turned to 180 degrees
- moved C2 10.8 mm to (25.4, 35.6)
- moved BAT1 9.73 mm to (26.0, 19.7), turned to 90 degrees
- moved NP1 8.98 mm to (25.4, 25.4)
- moved C1 8.28 mm to (25.4, 29.2), turned to 0 degrees
- moved ATTINY85-1 7.82 mm to (25.4, 19.7)
- moved C5 7.10 mm to (15.2, 25.4), turned to 90 degrees
- moved NP3 6.84 mm to (39.4, 25.4), turned to 90 degrees
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Connections:
- net +3V3: now also BAT1.V+, ON/OFF.1; no longer BAT1.BAT+, SW2.1
- net BAT+: now also ON/OFF.2, ON/OFF.3; no longer SW2.2, SW2.3
- net GND: now also BAT1.V-; no longer BAT1.BAT-
- net PB3: now also H3.2
Routing:
- net +3V3: track 13.7 -> 45.1 mm
- net BAT+: track 63.8 -> 93.3 mm, vias 3 -> 1
- net N$9: track 0.00 -> 19.2 mm
- net N$6: track 0.00 -> 17.8 mm, vias 0 -> 2
- net N$8: track 0.00 -> 17.8 mm
- net N$7: track 0.00 -> 16.3 mm, vias 0 -> 2
- net PB3: track 11.4 -> 24.2 mm, vias 0 -> 1
- net N$4: track 25.1 -> 35.6 mm
- net N$5: track 15.2 -> 23.9 mm
- net N$1: track 7.81 -> 15.9 mm
- net N$3: track 15.9 -> 21.9 mm
- net N$2: track 15.9 -> 21.0 mm
Other:
- board size 32 x 32 mm -> 38 x 38 mm
- board text added: "ON"
- board text removed: "PCB4-SK68"
