File: BootLoader/BootLoader_ATmega32U4/bootloader1.brd (EAGLE design)
At the start: 100 x 80 mm, 8 parts, among them U1 ATTINY85-20P

Commit message: UPD: pcb4-SK6812/pcb4.pdf
Routing:
- net GND: track 48.3 -> 43.2 mm
Changed lines of the file:
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@@
 <contactref element="U1" pad="4"/>
 <contactref element="GND" pad="1"/>
-<contactref element="SV1" pad="4"/>
 <contactref element="GND2" pad="1"/>
 <via x="63.5" y="20.32" extent="1-16" drill="0.35"/>
-<wire x1="73.66" y1="17.78" x2="73.66" y2="20.32" width="0.6096" layer="1"/>
-<wire x1="73.66" y1="17.78" x2="71.12" y2="17.78" width="0.6096" layer="1"/>
 <wire x1="73.66" y1="20.32" x2="63.5" y2="20.32" width="0.6096" layer="1"/>
 <wire x1="63.5" y1="20.32" x2="33.02" y2="20.32" width="0.6096" layer="16"/>
 <wire x1="33.02" y1="17.78" x2="33.02" y2="20.32" width="0.6096" layer="16"/>
+<contactref element="SV1" pad="4"/>
+<wire x1="71.12" y1="17.78" x2="73.66" y2="17.78" width="0" layer="19" extent="1-1"/>
+<wire x1="73.66" y1="20.32" x2="73.66" y2="17.78" width="0" layer="19" extent="1-1"/>
 </signal>
 <signal name="PB4">
