File: ATTiny85/ATTiny85+CirleLEDs+CR2032/pcb/pcb2-KiCad/pcb2-3-KiCad/pcb2-3/pcb2-3.kicad_sch (KiCad schematic)
At the start: 11 parts, among them SW1 bat+, SW2 POWER, U1 ATtiny85-20S

Commit message: UPD: directory tree: pcb/
Parts:
- added J1: Conn_01x03_Socket, symbol Connector:Conn_01x03_Socket
Changed lines of the file:
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@@
+	)
+	(symbol
+		(lib_id "Connector:Conn_01x03_Socket")
+		(at 114.3 148.59 0)
+		(unit 1)
+		(exclude_from_sim no)
+		(in_bom yes)
+		(on_board yes)
+		(dnp no)
+		(fields_autoplaced yes)
+		(property "Reference" "J1"
+			(at 115.57 147.3199 0)
+			(effects
+				(font
+					(size 1.27 1.27)
+				)
+				(justify left)
+			)
+		)
+		(property "Value" "Conn_01x03_Socket"
+			(at 115.57 149.8599 0)
+			(effects
+				(font
+					(size 1.27 1.27)
+				)
+				(justify left)
+			)
+		)
+		(property "Footprint" ""
+			(at 114.3 148.59 0)
+			(effects
+				(font
+					(size 1.27 1.27)
+				)
+				(hide yes)
+			)
+		)
+		(property "Datasheet" "~"
+			(at 114.3 148.59 0)
+			(effects
+				(font
+					(size 1.27 1.27)
+				)
+				(hide yes)
+			)
+		)
+		(property "Description" "Generic connector, single row, 01x03, script generated"
+			(at 114.3 148.59 0)
+			(effects
+				(font
+					(size 1.27 1.27)
+				)
+				(hide yes)
+			)
+		)
+		(pin "1"
+		)
+		(pin "3"
+		)
+		(pin "2"
+		)
+		(instances
+			(project ""
+				(path "/81b8b084-8461-4b3c-ac30-62ddc960295f"
+					(reference "J1")
+					(unit 1)
+				)
+			)
+		)
 	)
 	(symbol
